File: board/attiny/battery.kicad_pcb (KiCad board)
At the start: 2 copper layers, 17.8 x 26 mm, 10 parts, among them J1 Conn_01x06_Male, J2 Conn_01x02_Male, U1 ATtiny85-20SU, U2 LD1117S33TR_SOT223

Commit message: dev board
Other:
- net class Default removed
