File: board/bq3060/bq3060.kicad_pcb (KiCad board)
At the start: 2 copper layers, 74.2 x 52.8 mm, 70 parts, among them J1 Conn_01x04_Male, J2 Conn_01x03_Male, J3 Conn_01x03_Male, J4 Conn_01x03_Male, J5 Conn_01x02_Male, Q1 Si1023x, Q2 Si1023x, Q3 NDS351AN, Q4 SI4435DYTRPBF, Q5 SI4435DYTRPBF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

Commit message: dev board
Other:
- net class Default removed
